File: hardware/picoslidertoy/picoslidertoy.kicad_pcb (KiCad board)
At the start: 2 copper layers, 165.1 x 76.2 mm, 44 parts, among them SW1 Capacitive Button, SW2 Capacitive Button, SW3 Capacitive Button, SW4 Capacitive Button, SW5 Capacitive Button, SW6 Capacitive Button, SW7 Capacitive Button, SW8 Capacitive Button, U1 Pico

Commit message: pcb fixes
Parts:
- added H5: MountingHole, MountingHole:MountingHole_2.1mm, F.Cu at (82.2, 60.5)
- added H6: MountingHole, MountingHole:MountingHole_2.1mm, F.Cu at (105.8, 60.5)
- added H7: MountingHole, MountingHole:MountingHole_2.1mm, F.Cu at (82.2, 36.6)
- added H8: MountingHole, MountingHole:MountingHole_2.1mm, F.Cu at (105.8, 36.6)
Routing:
- net +3V3: track 140.5 -> 138.8 mm
- net /ROT2C: track 138.1 -> 136.5 mm
- net /ROT1C: track 107.8 -> 106.2 mm
- net /FADER2A: track 19.0 -> 17.8 mm
- net /TPAD2: track 41.4 -> 42.4 mm
- net /TPAD4: track 59.1 -> 58.0 mm
- net /TPAD3: track 42.2 -> 41.3 mm
- net /FADER3A: track 46.7 -> 47.6 mm
- net /ROT1B: track 104.4 -> 103.7 mm
- net /TPAD5: track 75.1 -> 74.5 mm
- net /ROT2B: track 143.7 -> 144.3 mm
- net /TPAD1: track 59.9 -> 59.4 mm

Commit message: pcb silksreen
Parts:
- removed R50, R51: 10k, Resistor_SMD:R_0603_1608Metric
- added R24: 1M, Resistor_SMD:R_0603_1608Metric, B.Cu at (109.2, 69.0)
- added R25: 10k, Resistor_SMD:R_0603_1608Metric, B.Cu at (111.3, 34.5)
- added R26: 10k, Resistor_SMD:R_0603_1608Metric, B.Cu at (115.6, 34.5)
- added SW9: Capacitive Button, SparkFun-Switch:Pad-CapacitiveTouch, F.Cu at (94.1, 63.5)
Connections:
- U1 pad 14: unconnected-(U1-GPIO10-Pad14) -> /ROT2A
- U1 pad 15: /ROT2A -> /ROT2B
- U1 pad 16: /ROT2B -> /ROT2C
- U1 pad 17: /ROT2C -> /TPAD9
Routing:
- net /TPAD9: track 0.00 -> 59.5 mm, vias 0 -> 2
- net /ROT2C: track 136.5 -> 138.4 mm
- net /ROT2B: track 144.3 -> 145.9 mm
- net /ROT2A: track 156.2 -> 157.5 mm
Other:
- board text added: "*"
- board text added: "1"
- board text added: "2"
- board text added: "3"
- board text added: "4"
- board text added: "5"
- board text added: "6"
- board text added: "7"
- board text added: "8"
- board text added: "@todbot"
- board text added: "picoslidertoy"
- board text added: "picoslidertoy github.com/todbot/picoslidertoy U1: Raspberry Pi Pico DISP1: 1.09{dblquote} I2C OLED SSD1306 R1-R23: 1M R25,R26: 10k"

Commit message: pcb proto submitted to fab
Other:
- board text added: "< >"
- board text added: "A"
- board text added: "B"
- board text added: "C"
- board text added: "JOCJLCJLCJLC"
- board text added: "X"
- board text added: "Y"
Changed lines of the file:
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@@
 			(unlocked yes)
 			(layer "F.SilkS")
+			(hide yes)
 			(effects
 				(font
@@
 		(attr smd)
 		(fp_text user "${REFERENCE}"
-			(at -0.5 -21.2 0)
+			(at -0.5 -22.098 0)
 			(unlocked yes)
 			(layer "F.Fab")
@@
 			(unlocked yes)
 			(layer "F.SilkS")
+			(hide yes)
 			(effects
 				(font
@@
 		(attr smd)
 		(fp_text user "${REFERENCE}"
-			(at -1.8 21.4 0)
+			(at -0.508 -22.098 0)
 			(unlocked yes)
 			(layer "F.Fab")
@@
 			(unlocked yes)
 			(layer "F.SilkS")
+			(hide yes)
 			(effects
 				(font
@@
 		(attr smd)
 		(fp_text user "${REFERENCE}"
-			(at -1.8 21.4 0)
+			(at -0.254 -22.098 0)
 			(unlocked yes)
 			(layer "F.Fab")
@@
 	)
 	(gr_circle
+		(center 168.91 55.88)
+		(end 173.99 55.88)
+		(stroke
+			(width 0.254)
+			(type default)
+		)
+		(fill none)
+		(layer "F.SilkS")
+	)
+	(gr_circle
 		(center 168.91 55.876893)
 		(end 186.69 55.876893)
@@
 		(layer "F.SilkS")
 	)
+	(gr_circle
+		(center 129.54 55.88)
+		(end 134.62 55.88)
+		(stroke
+			(width 0.254)
+			(type default)
+		)
+		(fill none)
+		(layer "F.SilkS")
+	)
 	(gr_arc
 		(start 59.566738 74.106369)
@@
 	)
 	(gr_line
-		(start 25.4 55.88)
-		(end 190.5 55.88)
-		(stroke
-			(width 0.1)
-			(type default)
-		)
-		(layer "Dwgs.User")
-	)
-	(gr_line
 		(start 30.48 25.4)
 		(end 185.42 25.4)
@@
 		(layer "Edge.Cuts")
 	)
+	(gr_text "JOCJLCJLCJLC"
+		(at 46.355 97.028 0)
+		(layer "B.SilkS")
+		(effects
+			(font
+				(size 1 1)
+				(thickness 0.1)
+			)
+			(justify left bottom mirror)
+		)
+	)
 	(gr_text "picoslidertoy\ngithub.com/todbot/picoslidertoy\nU1: Raspberry Pi Pico\nDISP1: 1.09{dblquote} I2C OLED SSD1306\nR1-R23: 1M\nR25,R26: 10k"
 		(at 154.432 71.882 0)
@@
 		)
 	)
+	(gr_text "A"
+		(at 35.56 56.896 0)
+		(layer "F.SilkS")
+		(effects
+			(font
+				(size 3.81 3.81)
+				(thickness 0.762)
+				(bold yes)
+			)
+			(justify left bottom)
+		)
+	)
 	(gr_text "8"
 		(at 173.228 88.646 0)
@@
 		)
 	)
+	(gr_text "B"
+		(at 52.07 56.896 0)
+		(layer "F.SilkS")
+		(effects
+			(font
+				(size 3.81 3.81)
+				(thickness 0.762)
+				(bold yes)
+			)
+			(justify left bottom)
+		)
+	)
+	(gr_text "<    >"
+		(at 111.633 57.785 0)
+		(layer "F.SilkS")
+		(effects
+			(font
+				(size 3.81 6.35)
+				(thickness 0.381)
+				(bold yes)
+			)
+			(justify left bottom)
+		)
+	)
 	(gr_text "7"
 		(at 154.178 88.392 0)
@@
 	)
 	(gr_text "picoslidertoy"
-		(at 141.986 31.75 0)
+		(at 141.986 33.274 0)
 		(layer "F.SilkS")
 		(effects
@@
 		(effects
 			(font
-				(size 2.54 2.54)
+				(size 1.27 2.54)
 				(thickness 0.254)
 			)
@@
 		)
 	)
+	(gr_text "X"
+		(at 127.254 58.42 0)
+		(layer "F.SilkS")
+		(effects
+			(font
+				(size 3.81 3.81)
+				(thickness 0.762)
+				(bold yes)
+			)
+			(justify left bottom)
+		)
+	)
+	(gr_text "Y"
+		(at 166.878 58.42 0)
+		(layer "F.SilkS")
+		(effects
+			(font
+				(size 3.81 3.81)
+				(thickness 0.762)
+				(bold yes)
+			)
+			(justify left bottom)
+		)
+	)
+	(gr_text "<    >"
+		(at 171.281725 73.732488 90)
+		(layer "F.SilkS")
+		(effects
+			(font
+				(size 3.81 6.35)
+				(thickness 0.381)
+				(bold yes)
+			)
+			(justify left bottom)
+		)
+	)
 	(gr_text "3"
-		(at 78.232 88.646 0)
+		(at 77.978 88.646 0)
+		(layer "F.SilkS")
+		(effects
+			(font
+				(size 3.81 3.81)
+				(thickness 0.762)
+				(bold yes)
+			)
+			(justify left bottom)
+		)
+	)
+	(gr_text "<     >"
+		(at 56.388 74.93 90)
+		(layer "F.SilkS")
+		(effects
+			(font
+				(size 3.81 6.35)
+				(thickness 0.381)
+				(bold yes)
+			)
+			(justify left bottom)
+		)
+	)
+	(gr_text "C"
+		(at 68.834 56.896 0)
 		(layer "F.SilkS")
 		(effects
@@
 		)
 	)
+	(gr_text "<    >"
+		(at 131.911725 73.732488 90)
+		(layer "F.SilkS")
+		(effects
+			(font
+				(size 3.81 6.35)
+				(thickness 0.381)
+				(bold yes)
+			)
+			(justify left bottom)
+		)
+	)
+	(gr_text "<    >"
+		(at 151.003 57.785 0)
+		(layer "F.SilkS")
+		(effects
+			(font
+				(size 3.81 6.35)
+				(thickness 0.381)
+				(bold yes)
+			)
+			(justify left bottom)
+		)
+	)
 	(gr_text "4"
-		(at 97.028 88.646 0)
+		(at 96.774 88.646 0)
 		(layer "F.SilkS")
 		(effects
@@
 		)
 	)
+	(gr_text "<     >"
+		(at 39.878 74.93 90)
+		(layer "F.SilkS")
+		(effects
+			(font
+				(size 3.81 6.35)
+				(thickness 0.381)
+				(bold yes)
+			)
+			(justify left bottom)
+		)
+	)
 	(gr_text "*"
 		(at 92.202 66.802 0)
@@
 				(bold yes)
 			)
+			(justify left bottom)
+		)
+	)
+	(gr_text "<     >"
+		(at 73.152 74.676 90)
+		(layer "F.SilkS")
+		(effects
+			(font
+				(size 3.81 6.35)
+				(thickness 0.381)
+				(bold yes)
+			)
