File: hardware/picoslidertoy/picoslidertoy.kicad_sch (KiCad schematic)
At the start: 44 parts, among them SW1 Capacitive Button, SW2 Capacitive Button, SW3 Capacitive Button, SW4 Capacitive Button, SW5 Capacitive Button, SW6 Capacitive Button, SW7 Capacitive Button, SW8 Capacitive Button, U1 Pico

Commit message: pcb fixes
Parts:
- added H5, H6, H7, H8: MountingHole, MountingHole:MountingHole_2.1mm, symbol Mechanical:MountingHole
Connections:
- no-connect marks 0 -> 8
Other:
- moved on the sheet: FADER1, FADER2, FADER3, H1, H2, H3, H4, R1, R10, R11, R12, R13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

Commit message: pcb silksreen
Parts:
- added R24: 1M, Resistor_SMD:R_0603_1608Metric, symbol Device:R
- added SW9: Capacitive Button, SparkFun-Switch:Pad-CapacitiveTouch, symbol SparkFun-Switch:Capacitive Button
- renumbered R51 to R25, R50 to R26
Connections:
- net GND: now also R24.1
- net ROT2A: now also U1.14 (GPIO10); no longer U1.15 (GPIO11)
- net ROT2B: now also U1.15 (GPIO11); no longer U1.16 (GPIO12)
- net ROT2C: now also U1.16 (GPIO12); no longer U1.17 (GPIO13)
- new net TPAD9: R24.2, SW9.1 (A), U1.17 (GPIO13)
Changed lines of the file:
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@@
 	(wire
 		(pts
-			(xy 26.67 83.82) (xy 39.37 83.82)
-		)
-		(stroke
-			(width 0)
-			(type default)
-		)
-	)
-	(wire
-		(pts
 			(xy 26.67 60.96) (xy 39.37 60.96)
 		)
@@
 	(wire
 		(pts
-			(xy 26.67 81.28) (xy 39.37 81.28)
-		)
-		(stroke
-			(width 0)
-			(type default)
-		)
-	)
-	(wire
-		(pts
 			(xy 26.67 73.66) (xy 39.37 73.66)
 		)
@@
 	(wire
 		(pts
-			(xy 26.67 78.74) (xy 39.37 78.74)
+			(xy 26.67 81.28) (xy 39.37 81.28)
 		)
 		(stroke
@@
 	(wire
 		(pts
+			(xy 26.67 83.82) (xy 39.37 83.82)
+		)
+		(stroke
+			(width 0)
+			(type default)
+		)
+	)
+	(wire
+		(pts
 			(xy 76.2 55.88) (xy 74.93 55.88)
 		)
@@
 	(wire
 		(pts
-			(xy 26.67 86.36) (xy 39.37 86.36)
+			(xy 140.97 85.09) (xy 154.94 85.09)
 		)
 		(stroke
@@
 	(wire
 		(pts
+			(xy 26.67 86.36) (xy 39.37 86.36)
+		)
+		(stroke
+			(width 0)
+			(type default)
+		)
+	)
+	(wire
+		(pts
 			(xy 132.08 31.75) (xy 133.35 31.75)
 		)
@@
 		)
 	)
+	(wire
+		(pts
+			(xy 26.67 78.74) (xy 39.37 78.74)
+		)
+		(stroke
+			(width 0)
+			(type default)
+		)
+	)
 	(label "FADER2A"
 		(at 213.36 67.31 0)
@@
 		)
 	)
+	(label "ROT2C"
+		(at 26.67 83.82 0)
+		(fields_autoplaced yes)
+		(effects
+			(font
+				(size 1.27 1.27)
+			)
+			(justify left bottom)
+		)
+	)
 	(label "TPAD6"
 		(at 82.55 91.44 0)
@@
 		)
 	)
-	(label "TPAD2"
-		(at 82.55 78.74 0)
+	(label "TPAD9"
+		(at 26.67 86.36 0)
 		(fields_autoplaced yes)
 		(effects
@@
 		)
 	)
-	(label "TPAD1"
-		(at 82.55 73.66 0)
+	(label "TPAD2"
+		(at 82.55 78.74 0)
 		(fields_autoplaced yes)
 		(effects
@@
 		)
 	)
-	(label "TPAD4"
-		(at 144.78 50.8 0)
+	(label "TPAD1"
+		(at 82.55 73.66 0)
 		(fields_autoplaced yes)
 		(effects
@@
 		)
 	)
-	(label "ROT2C"
-		(at 215.9 154.94 0)
+	(label "TPAD4"
+		(at 144.78 50.8 0)
 		(fields_autoplaced yes)
 		(effects
@@
 	)
 	(label "ROT2C"
-		(at 27.94 86.36 0)
+		(at 215.9 154.94 0)
 		(fields_autoplaced yes)
 		(effects
@@
 		)
 	)
+	(label "ROT2A"
+		(at 26.67 78.74 0)
+		(fields_autoplaced yes)
+		(effects
+			(font
+				(size 1.27 1.27)
+			)
+			(justify left bottom)
+		)
+	)
 	(label "FADER1A"
 		(at 213.36 40.64 0)
@@
 		)
 	)
-	(label "ROT2A"
-		(at 27.94 81.28 0)
-		(fields_autoplaced yes)
-		(effects
-			(font
-				(size 1.27 1.27)
-			)
-			(justify left bottom)
-		)
-	)
 	(label "FADER3A"
 		(at 213.36 93.98 0)
@@
 		)
 	)
+	(label "ROT2B"
+		(at 26.67 81.28 0)
+		(fields_autoplaced yes)
+		(effects
+			(font
+				(size 1.27 1.27)
+			)
+			(justify left bottom)
+		)
+	)
 	(label "ROT1A"
 		(at 26.67 68.58 0)
@@
 		)
 	)
+	(label "TPAD9"
+		(at 144.78 85.09 0)
+		(fields_autoplaced yes)
+		(effects
+			(font
+				(size 1.27 1.27)
+			)
+			(justify left bottom)
+		)
+	)
 	(label "TPAD7"
 		(at 144.78 72.39 0)
@@
 		)
 	)
-	(label "ROT2B"
-		(at 27.94 83.82 0)
-		(fields_autoplaced yes)
-		(effects
-			(font
-				(size 1.27 1.27)
-			)
-			(justify left bottom)
-		)
-	)
 	(symbol
 		(lib_id "Device:R")
@@
 		(on_board yes)
 		(dnp no)
-		(property "Reference" "R50"
+		(property "Reference" "R26"
 			(at 85.344 109.474 90)
 			(effects
@@
 			(project "picoslidertoy"
 				(path "/b1a19a0a-6a78-4edf-a179-1dffdce9f58b"
-					(reference "R50")
+					(reference "R26")
 					(unit 1)
 				)
@@
 		(on_board yes)
 		(dnp no)
-		(property "Reference" "R51"
+		(property "Reference" "R25"
 			(at 78.994 109.474 90)
 			(effects
@@
 			(project "picoslidertoy"
 				(path "/b1a19a0a-6a78-4edf-a179-1dffdce9f58b"
-					(reference "R51")
+					(reference "R25")
 					(unit 1)
 				)
@@
 	)
 	(symbol
+		(lib_id "Device:R")
+		(at 137.16 85.09 90)
+		(unit 1)
+		(exclude_from_sim no)
+		(in_bom yes)
+		(on_board yes)
+		(dnp no)
+		(property "Reference" "R24"
+			(at 135.636 82.804 90)
+			(effects
+				(font
+					(size 1.27 1.27)
+				)
+			)
+		)
+		(property "Value" "1M"
+			(at 138.43 87.122 90)
+			(effects
+				(font
+					(size 1.27 1.27)
+				)
+			)
+		)
+		(property "Footprint" "Resistor_SMD:R_0603_1608Metric"
+			(at 137.16 86.868 90)
+			(effects
+				(font
+					(size 1.27 1.27)
+				)
+				(hide yes)
+			)
+		)
+		(property "Datasheet" "~"
+			(at 137.16 85.09 0)
+			(effects
+				(font
+					(size 1.27 1.27)
+				)
+				(hide yes)
+			)
+		)
+		(property "Description" "Resistor"
+			(at 137.16 85.09 0)
+			(effects
+				(font
+					(size 1.27 1.27)
+				)
+				(hide yes)
+			)
+		)
+		(pin "2"
+		)
+		(pin "1"
+		)
+		(instances
+			(project "picoslidertoy"
+				(path "/b1a19a0a-6a78-4edf-a179-1dffdce9f58b"
+					(reference "R24")
+					(unit 1)
+				)
+			)
+		)
+	)
+	(symbol
 		(lib_id "power:GND")
 		(at 132.08 38.1 270)
@@
 	)
 	(symbol
+		(lib_id "SparkFun-Switch:Capacitive Button")
+		(at 154.94 85.09 270)
+		(unit 1)
+		(exclude_from_sim no)
+		(in_bom yes)
+		(on_board yes)
+		(dnp no)
+		(fields_autoplaced yes)
+		(property "Reference" "SW9"
+			(at 160.02 83.8199 90)
+			(effects
+				(font
+					(size 1.27 1.27)
+				)
+				(justify left)
+			)
+		)
+		(property "Value" "Capacitive Button"
+			(at 160.02 86.3599 90)
+			(effects
+				(font
+					(size 1.27 1.27)
+				)
+				(justify left)
+			)
+		)
+		(property "Footprint" "SparkFun-Switch:Pad-CapacitiveTouch"
+			(at 147.32 85.09 0)
+			(effects
+				(font
+					(size 1.27 1.27)
+				)
+				(hide yes)
+			)
+		)
+		(property "Datasheet" "~"
+			(at 144.78 85.09 0)
+			(effects
+				(font
+					(size 1.27 1.27)
+				)
+				(hide yes)
+			)
+		)
+		(property "Description" "Single Pole Single Throw (SPST) switch"
+			(at 154.94 85.09 0)
+			(effects
+				(font
+					(size 1.27 1.27)
+				)
+				(hide yes)
+			)
+		)
+		(pin "1"
+		)
+		(instances
+			(project "picoslidertoy"
+				(path "/b1a19a0a-6a78-4edf-a179-1dffdce9f58b"
+					(reference "SW9")
+					(unit 1)
+				)
+			)
+		)
+	)
+	(symbol
 		(lib_id "power:GND")
 		(at 203.2 154.94 270)
@@
 					(unit 1)
 				)
+			)
+		)
+	)
+	(symbol
+		(lib_id "power:GND")
+		(at 133.35 85.09 270)
+		(unit 1)
+		(exclude_from_sim no)
+		(in_bom yes)
+		(on_board yes)
+		(dnp no)
+		(fields_autoplaced yes)
+		(property "Reference" "#PWR036"
+			(at 127 85.09 0)
+			(effects
+				(font
+					(size 1.27 1.27)
+				)
+				(hide yes)
+			)
+		)
+		(property "Value" "GND"
+			(at 129.54 85.0899 90)
+			(effects
+				(font
+					(size 1.27 1.27)
+				)
+				(justify right)
+			)
+		)
+		(property "Footprint" ""
+			(at 133.35 85.09 0)
+			(effects
+				(font
+					(size 1.27 1.27)
+				)
+				(hide yes)
+			)
+		)
+		(property "Datasheet" ""
+			(at 133.35 85.09 0)
+			(effects
+				(font
+					(size 1.27 1.27)
+				)
+				(hide yes)
+			)
+		)
+		(property "Description" "Power symbol creates a global label with name \"GND\" , ground"
+			(at 133.35 85.09 0)
+			(effects
+				(font
+					(size 1.27 1.27)
+				)
+				(hide yes)
+			)
+		)
+		(pin "1"
+		)
+		(instances
+			(project "picoslidertoy"
+				(path "/b1a19a0a-6a78-4edf-a179-1dffdce9f58b"
+					(reference "#PWR036")
+					(unit 1)
+				)

Commit message: pcb display positioning tune
Parts:
- removed DISP1: HS96L03W2C03, todbot_stuff:OLED-TH_under_L27.8-W27.2-P2.54_C9900033791, symbol easyeda2kicad:HS96L03W2C03
- added DISP2: HS96L03W2C03, todbot_stuff:OLED-TH_under_fixed_L27.8-W27.2-P2.54_C9900033791, symbol easyeda2kicad:HS96L03W2C03
- H5, H7, H8: footprint MountingHole:MountingHole_2.1mm -> MountingHole:MountingHole_2.5mm
- H6: footprint MountingHole:MountingHole_2.1mm -> MountingHole:MountingHole_2.7mm
Connections:
- net +3V3: now also DISP2.2 (VCC)
- net GND: now also DISP2.1 (GND)
- net SCL: now also DISP2.3 (SCL)
- net SDA: now also DISP2.4 (SDA)
Changed lines of the file:
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@@
 			)
 		)
-		(property "Footprint" "MountingHole:MountingHole_2.1mm"
+		(property "Footprint" "MountingHole:MountingHole_2.5mm"
 			(at 156.21 181.61 0)
 			(effects
@@
 			)
 		)
-		(property "Footprint" "MountingHole:MountingHole_2.1mm"
+		(property "Footprint" "MountingHole:MountingHole_2.5mm"
 			(at 156.21 171.45 0)
 			(effects
@@
 			)
 		)
-		(property "Footprint" "MountingHole:MountingHole_2.1mm"
+		(property "Footprint" "MountingHole:MountingHole_2.7mm"
 			(at 156.21 176.53 0)
 			(effects
@@
 	)
 	(symbol
-		(lib_id "easyeda2kicad:HS96L03W2C03")
-		(at 96.52 116.84 0)
-		(mirror x)
-		(unit 1)
-		(exclude_from_sim no)
-		(in_bom yes)
-		(on_board yes)
-		(dnp no)
-		(property "Reference" "DISP1"
-			(at 101.6 118.1101 0)
-			(effects
-				(font
-					(size 1.27 1.27)
-				)
-				(justify left)
-			)
-		)
-		(property "Value" "HS96L03W2C03"
-			(at 101.6 115.5701 0)
-			(effects
-				(font
-					(size 1.27 1.27)
-				)
-				(justify left)
-			)
-		)
-		(property "Footprint" "todbot_stuff:OLED-TH_under_L27.8-W27.2-P2.54_C9900033791"
-			(at 96.52 105.41 0)
-			(effects
-				(font
-					(size 1.27 1.27)
-				)
-				(hide yes)
-			)
-		)
-		(property "Datasheet" ""
-			(at 96.52 116.84 0)
-			(effects
-				(font
-					(size 1.27 1.27)
-				)
-				(hide yes)
-			)
-		)
-		(property "Description" ""
-			(at 96.52 116.84 0)
-			(effects
-				(font
-					(size 1.27 1.27)
-				)
-				(hide yes)
-			)
-		)
-		(property "LCSC Part" "C5248080"
-			(at 96.52 102.87 0)
-			(effects
-				(font
-					(size 1.27 1.27)
-				)
-				(hide yes)
-			)
-		)
-		(pin "3"
-		)
-		(pin "2"
-		)
-		(pin "4"
-		)
-		(pin "1"
-		)
-		(instances
-			(project "picoslidertoy"
-				(path "/b1a19a0a-6a78-4edf-a179-1dffdce9f58b"
-					(reference "DISP1")
-					(unit 1)
-				)
-			)
-		)
-	)
-	(symbol
 		(lib_id "SparkFun-Switch:Capacitive Button")
 		(at 154.94 50.8 270)
@@
 			)
 		)
-		(property "Footprint" "MountingHole:MountingHole_2.1mm"
+		(property "Footprint" "MountingHole:MountingHole_2.5mm"
 			(at 156.21 186.69 0)
 			(effects
@@
 					(unit 1)
 				)
+			)
+		)
+	)
+	(symbol
+		(lib_id "easyeda2kicad:HS96L03W2C03")
+		(at 96.52 116.84 0)
+		(mirror x)
+		(unit 1)
+		(exclude_from_sim no)
+		(in_bom yes)
+		(on_board yes)
+		(dnp no)
+		(property "Reference" "DISP2"
+			(at 101.6 118.1101 0)
+			(effects
+				(font
+					(size 1.27 1.27)
+				)
+				(justify left)
+			)
+		)
+		(property "Value" "HS96L03W2C03"
+			(at 101.6 115.5701 0)
+			(effects
+				(font
+					(size 1.27 1.27)
+				)
+				(justify left)
+			)
+		)
+		(property "Footprint" "todbot_stuff:OLED-TH_under_fixed_L27.8-W27.2-P2.54_C9900033791"
+			(at 96.52 105.41 0)
+			(effects
+				(font
+					(size 1.27 1.27)
+				)
+				(hide yes)
+			)
+		)
+		(property "Datasheet" ""
+			(at 96.52 116.84 0)
+			(effects
+				(font
+					(size 1.27 1.27)
+				)
+				(hide yes)
+			)
+		)
+		(property "Description" ""
+			(at 96.52 116.84 0)
+			(effects
+				(font
+					(size 1.27 1.27)
+				)
+				(hide yes)
+			)
+		)
+		(property "LCSC Part" "C5248080"
+			(at 96.52 102.87 0)
+			(effects
+				(font
+					(size 1.27 1.27)
+				)
+				(hide yes)
+			)
+		)
+		(pin "3"
+		)
+		(pin "2"
+		)
+		(pin "4"
+		)
+		(pin "1"
+		)
+		(instances
+			(project "picoslidertoy"
+				(path "/b1a19a0a-6a78-4edf-a179-1dffdce9f58b"
+					(reference "DISP2")
+					(unit 1)
+				)

Commit message: pcb display position tuning
Parts:
- removed H5, H7, H8: MountingHole, MountingHole:MountingHole_2.5mm, symbol Mechanical:MountingHole
- removed H6: MountingHole, MountingHole:MountingHole_2.7mm, symbol Mechanical:MountingHole
- renumbered DISP2 to DISP1
