File: schematics/picoslidertoy/picoslidertoy.kicad_pcb (KiCad board)
At the start: 2 copper layers, 165.1 x 76.2 mm, 46 parts, among them SW1 Capacitive Button, SW2 Capacitive Button, SW3 Capacitive Button, SW4 Capacitive Button, SW5 Capacitive Button, SW6 Capacitive Button, SW7 Capacitive Button, SW8 Capacitive Button, SW9 Capacitive Button, U1 Pico

Commit message: new display hole-less pcb to fab
Other:
- board text added: "picoslidertoy github.com/todbot/picoslidertoy U1: Raspberry Pi Pico DISP1: 0.96{dblquote} I2C OLED display SSD1306 R1-R24: 1M R25,R26: 10k 24 Apr 2024 - (no display mounting holes)"
- board text removed: "picoslidertoy github.com/todbot/picoslidertoy U1: Raspberry Pi Pico DISP1: 0.96{dblquote} I2C OLED SSD1306 R1-R24: 1M R25,R26: 10k 24 Apr 2024 - (no display mounting holes)"
Changed lines of the file:
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@@
 		)
 	)
-	(gr_text "picoslidertoy\ngithub.com/todbot/picoslidertoy\nU1: Raspberry Pi Pico\nDISP1: 0.96{dblquote} I2C OLED SSD1306\nR1-R24: 1M\nR25,R26: 10k\n24 Apr 2024 - (no display mounting holes)"
+	(gr_text "picoslidertoy\ngithub.com/todbot/picoslidertoy\nU1: Raspberry Pi Pico\nDISP1: 0.96{dblquote} I2C OLED display SSD1306\nR1-R24: 1M\nR25,R26: 10k\n24 Apr 2024 - (no display mounting holes)"
 		(at 154.432 71.882 0)
 		(layer "B.SilkS")
